File: EltekController/EltekController.kicad_pcb (KiCad board)
At the start: 2 copper layers, 57.5 x 45 mm, 36 parts, among them J1 CANBUS, J2 Display, Q1 UMH3N, U1 ESP32-WROOM-32E, U2 CP2104-F03-GMR, U3 TJA1051T/3/1J, U4 AMS1117-3.3

Commit message: saving this because I changed my mind again
Parts:
- removed the C7 at (127.4, 114.8)
- removed the C8 at (123.6, 108.2)
- removed the D2 at (148.5, 118.5)
- removed PS1: SPBW06G-05, SnapEDA-zip:CONV_SPBW06F-12
- removed Q1: UMH3N, Package_TO_SOT_SMD:SOT-363_SC-70-6
- removed RN1: 1K, Resistor_SMD:R_Array_Concave_4x0402
- added C1: 10uF, Capacitor_SMD:C_0603_1608Metric, F.Cu at (245.6, 84.8)
- added C10: 100nF, Capacitor_SMD:C_0402_1005Metric, F.Cu at (245.1, 87.1)
- added C3: 2.2uF, Capacitor_SMD:C_1210_3225Metric_Pad1.33x2.70mm_HandSolder, F.Cu at (109.4, 108.9)
- added C5: 22uF, Capacitor_SMD:C_0805_2012Metric, F.Cu at (116.7, 104.9)
- added C9: 100nF, Capacitor_SMD:C_0402_1005Metric, F.Cu at (242.0, 89.6)
- added D1: SS210, Diode_SMD:D_PowerDI-123, F.Cu at (113.4, 106.3)
- added D3: RGB, 1 My Footprints:DY-S1515065_RGBC_6805-5T, F.Cu at (239.8, 86.0)
- added D4: 3V3, 1 My Footprints:LED_0603_1608Metric_SnapModel, F.Cu at (253.9, 104.7)
- added J3: ESP_PROG, 1 My Footprints:JST_SH_SM06B-SRSS-TB_1x06-1MP_P1.00mm_Horizontal_3D, F.Cu at (201.6, 75.2)
- added JP1: VPP_EN, Jumper:SolderJumper-2_P1.3mm_Open_RoundedPad1.0x1.5mm, F.Cu at (219.5, 107.0)
- added L1: 33uH, 1 My Footprints:L_Sunlord_SWPA6028S, F.Cu at (115.0, 100.0)
- added PS: Converter_DCDC_TDK-Lambda_CC3-xxxxxF-E, 1 My Footprints:Converter_DCDC_TDK-Lambda_CC3-xxxxxF-E, F.Cu at (86.0, 86.2)
- added R2: 68K, Resistor_SMD:R_0402_1005Metric, F.Cu at (108.4, 96.4)
- added R3: 12K, Resistor_SMD:R_0402_1005Metric, F.Cu at (108.4, 97.6)
- added R5: 22R, Resistor_SMD:R_0402_1005Metric, F.Cu at (227.2, 102.3)
- added R6: 1K, Resistor_SMD:R_0402_1005Metric, F.Cu at (230.9, 99.7)
- added R7: 1K, Resistor_SMD:R_0402_1005Metric, F.Cu at (239.2, 89.6)
- C2: value 10uF -> 100nF; footprint Capacitor_SMD:C_0603_1608Metric -> Capacitor_SMD:C_0402_1005Metric
- C4: renamed from C10; value 1uF -> 2.2uF; footprint Capacitor_SMD:C_1206_3216Metric -> Capacitor_SMD:C_1210_3225Metric_Pad1.33x2.70mm_HandSolder
- C6: value 1uF -> 22uF; footprint Capacitor_SMD:C_0402_1005Metric -> Capacitor_SMD:C_0805_2012Metric
- D5: renamed from D3; value IO2 -> 5V0
- I2C1: footprint Connector_PinSocket_2.54mm:PinSocket_1x04_P2.54mm_Vertical -> 1 My Footprints:OLED_SSD1315_128x64_1.3_I2C_New_Silhouette
- U1: value ESP32-WROOM-32E -> ESP32-S2-WROVER; footprint 1 My Footprints:ESP32-WROOM_WROVER_Dual_JLC_ManyVias -> 1 My Footprints:ESP32-S2-WROVER_and_WROOM(PCB,-I(IPEX))-Universal
- U2: value CP2104-F03-GMR -> LMR16006XDDCR; footprint Package_DFN_QFN:QFN-24-1EP_4x4mm_P0.5mm_EP2.6x2.6mm -> Package_TO_SOT_SMD:SOT-23-6
- U3: value TJA1051T/3/1J -> MAX3051ESA
- USB1: value USB-SER -> USB-OTG
- moved USB1 106.2 mm to (231.9, 113.2)
- moved D2 90.2 mm to (202.2, 104.5)
- moved U3 89.4 mm to (218.8, 74.0)
- moved J2 87.9 mm to (194.2, 88.2)
- moved JP3 81.5 mm to (194.3, 115.8)
- moved D5 72.1 mm to (217.1, 123.8)
- moved S1 72.1 mm to (212.6, 123.8)
- moved S2 72.1 mm to (206.1, 123.8)
- moved C11 67.0 mm to (220.2, 83.9)
- moved C12 67.0 mm to (220.2, 85.7)
- moved R1 67.0 mm to (217.9, 85.5)
- moved I2C1 54.7 mm to (181.4, 49.0), turned to 0 degrees
- moved C14 45.2 mm to (126.9, 54.7)
- moved U4 45.2 mm to (122.3, 56.1)
- moved C6 39.2 mm to (116.7, 107.4), turned to 0 degrees
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- renumbered C4 to C11, C5 to C12, C3 to C14, C1 to C7, C9 to C8, D1 to D2, JP1 to JP2, JP2 to JP3, R2 to R1, R1 to R4, S2 to S1, S1 to S2
Connections:
- net Net-(USB1-Pad4) renamed /USB_ID
- C2 pad 1: GND -> /SW
- C2 pad 2: +5V -> /CB
- C4 pad 1: GNDPWR -> +48V
- C4 pad 2: +48V -> GND
- C6 pad 1: /~RST -> GND
- C6 pad 2: GND -> +5V
- C7 pad 1: +5V -> GND
- C7 pad 2: GND -> +3V3
- C8 pad 2: +5V -> GND
- D5 pad 2: +3V3 -> +5V
- NT1 pad 1: GND -> GNDPWR
- NT1 pad 2: GNDPWR -> GND
- U1 pad 10: /CAN_S -> /OLED_SCL
- U1 pad 11: /CAN_TX -> Net-(U1-Pad11)
- U1 pad 12: /CAN_RX -> Net-(U1-Pad12)
- U1 pad 14: Net-(U1-Pad14) -> /~CAN_EN
- U1 pad 15: GND -> /CAN_TX
- U1 pad 16: Net-(U1-Pad16) -> /CAN_RX
- U1 pad 22: Net-(U1-Pad22) -> /USB_D-
- U1 pad 23: Net-(U1-Pad23) -> /USB_D+
- U1 pad 24: /GPIO2_LED -> Net-(U1-Pad24)
- U1 pad 25: /~BOOT -> Net-(U1-Pad25)
- U1 pad 26: Net-(U1-Pad26) -> GND
- U1 pad 27: /D_RXSDA -> Net-(U1-Pad27)
- U1 pad 28: /D_TXSCL -> Net-(U1-Pad28)
- U1 pad 29: /LED_R -> Net-(U1-Pad29)
- U1 pad 3: /~RST -> /~BOOT
- U1 pad 30: /LED_G -> /LED_DAT
- U1 pad 31: /LED_B -> /D_TXSCL
- U1 pad 32: Net-(U1-Pad32) -> /D_RXSDA
- U1 pad 34: /UART_RX -> Net-(U1-Pad34)
- U1 pad 35: /UART_TX -> Net-(U1-Pad35)
- U1 pad 37: Net-(U1-Pad37) -> /UART_TX
- U1 pad 38: GND -> /UART_RX
- U1 pad 39: GND -> Net-(U1-Pad39)
- U1 pad 8: /OLED_SDA -> Net-(U1-Pad8)
- U1 pad 9: /OLED_SCL -> /OLED_SDA
- U2 pad 1: Net-(U2-Pad1) -> /CB
- U2 pad 3: /USB_D+ -> /FB
- U2 pad 4: /USB_D- -> Net-(U2-Pad4)
- U2 pad 5: +3V3 -> +48V
- U2 pad 6: +3V3 -> /SW
- U3 pad 3: +5V -> +3V3
- U3 pad 5: +3V3 -> /~CAN_EN
- U3 pad 8: /CAN_S -> GND
Routing:
- net +3V3: track 132.1 -> 0.00 mm, vias 11 -> 0
- net /~RST: track 58.0 -> 0.00 mm, vias 2 -> 0
- net +5V: track 51.6 -> 6.92 mm, vias 3 -> 0
- net /D_TXSCL: track 32.3 -> 0.00 mm, vias 1 -> 0
- net /D_RXSDA: track 30.2 -> 0.00 mm, vias 1 -> 0
- net /CAN-: track 26.8 -> 0.00 mm, vias 1 -> 0
- net /UART_TX: track 25.9 -> 0.00 mm, vias 2 -> 0
- net /UART_RX: track 25.3 -> 0.00 mm, vias 2 -> 0
- net /VBUS: track 23.9 -> 0.00 mm
- net /CAN+: track 21.5 -> 0.00 mm, vias 1 -> 0
- net /CAN_S: track 20.7 -> 0.00 mm
- net /CAN_TX: track 19.4 -> 0.00 mm
- net /~BOOT: track 17.6 -> 0.00 mm
- net /CAN_RX: track 14.5 -> 0.00 mm
- net GND: track 12.6 -> 0.00 mm, vias 67 -> 11
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- added copper zone on F.Cu, net +48V
- added copper zone on F.Cu, net +5V
- added copper zone on F.Cu, net /SW
- removed copper zone on B.Cu, net GNDPWR
- removed copper zone on F.Cu, net GNDPWR
Other:
- board size 57.5 x 45 mm -> 80 x 35 mm

Commit message: yes, good
Parts:
- removed C10: 100nF, Capacitor_SMD:C_0402_1005Metric
- removed the C11 at (220.2, 83.9)
- removed C12: 100nF, Capacitor_SMD:C_0603_1608Metric
- removed C14: 22uF, Capacitor_SMD:C_0603_1608Metric
- removed C5: 22uF, Capacitor_SMD:C_0805_2012Metric
- removed the D1 at (113.4, 106.3)
- removed D5: 5V0, 1 My Footprints:LED_0603_1608Metric_SnapModel
- removed JP3: VJ2, Jumper:SolderJumper-3_P1.3mm_Open_RoundedPad1.0x1.5mm_NumberLabels
- removed L1: 33uH, 1 My Footprints:L_Sunlord_SWPA6028S
- removed PS: Converter_DCDC_TDK-Lambda_CC3-xxxxxF-E, 1 My Footprints:Converter_DCDC_TDK-Lambda_CC3-xxxxxF-E
- removed R1: 10K, Resistor_SMD:R_0402_1005Metric
- removed R3: 12K, Resistor_SMD:R_0402_1005Metric
- removed the R4 at (142.8, 61.9)
- removed R5: 22R, Resistor_SMD:R_0402_1005Metric
- removed R7: 1K, Resistor_SMD:R_0402_1005Metric
- removed S1: Boot, 1 My Footprints:SW_Push_1P1T-SH_NO_CK_KMR2xxG_3D
- removed U4: AMS1117-3.3, Package_TO_SOT_SMD:SOT-223-3_TabPin2
- added C1: 10uF, Capacitor_SMD:C_0402_1005Metric, F.Cu at (135.2, 82.5)
- added PS1: CC3-4803SF-E, 1 My Footprints:Converter_DCDC_TDK-Lambda_CC3-xxxxxF-E, F.Cu at (113.8, 100.5)
- added R6: 10K, Resistor_SMD:R_0402_1005Metric, F.Cu at (108.8, 111.0)
- added R9: 120R, Resistor_SMD:R_0805_2012Metric_Pad1.15x1.40mm_HandSolder, F.Cu at (103.1, 88.2)
- added SW2: BOOT, 1 My Footprints:KEY-SMD_4P-L4.2-W3.2-P2.20-LS5.1-TL, F.Cu at (121.2, 111.0)
- added SW3: LEFT, 1 My Footprints:KEY-SMD_4P-L4.2-W3.2-P2.20-LS5.1-TL, F.Cu at (132.2, 111.0)
- added SW4: SEL, 1 My Footprints:KEY-SMD_4P-L4.2-W3.2-P2.20-LS5.1-TL, F.Cu at (141.7, 111.0)
- added SW5: RIGHT, 1 My Footprints:KEY-SMD_4P-L4.2-W3.2-P2.20-LS5.1-TL, F.Cu at (151.2, 111.0)
- C2: value 100nF -> 10uF
- C3: value 2.2uF -> 10uF; footprint Capacitor_SMD:C_1210_3225Metric_Pad1.33x2.70mm_HandSolder -> Capacitor_SMD:C_0402_1005Metric
- C4: value 2.2uF -> 22uF; footprint Capacitor_SMD:C_1210_3225Metric_Pad1.33x2.70mm_HandSolder -> Capacitor_SMD:C_0603_1608Metric
- C6: value 22uF -> 100nF; footprint Capacitor_SMD:C_0805_2012Metric -> Capacitor_SMD:C_0402_1005Metric
- C7: value 10uF -> 100nF; footprint Capacitor_SMD:C_0603_1608Metric -> Capacitor_SMD:C_0402_1005Metric
- D1: renamed from D4; value 3V3 -> IO2
- D2: value B5819W -> PWR; footprint Diode_SMD:D_SOD-123 -> 1 My Footprints:LED_0603_1608Metric_SnapModel
- D3: value RGB -> SK6812MINI; footprint 1 My Footprints:DY-S1515065_RGBC_6805-5T -> 1 My Footprints:LED_SK6812MINI_PLCC4_3.5x3.5mm_P1.75mm_3D
- H1, H2, H3, H4: footprint MountingHole:MountingHole_2.7mm_M2.5_Pad_Via -> MountingHole:MountingHole_2.7mm_M2.5_ISO7380_Pad_TopBottom
- I2C1: footprint 1 My Footprints:OLED_SSD1315_128x64_1.3_I2C_New_Silhouette -> 1 My Footprints:OLED_SSD1315_128x64_1.3_I2C_New_Silhouette_Big3D
- J1: footprint 1 My Footprints:Molex_Nano-Fit_105309-xx04_1x04_P2.50mm_Vertical_Horizontal_Combined -> SnapEDA-zip:TE_5-103634-3
- J2: value Display -> Conn_01x06; footprint Connector_JST:JST_XH_S4B-XH-A_1x04_P2.50mm_Horizontal -> ESP32-S2-DevKit-USB-Rev-B:WU06S
- J3: value ESP_PROG -> Qwiic; footprint 1 My Footprints:JST_SH_SM06B-SRSS-TB_1x06-1MP_P1.00mm_Horizontal_3D -> 1 My Footprints:JST_SH_SM04B-SRSS-TB_1x04-1MP_P1.00mm_Horizontal_3D
- JP2: moved to F.Cu
- R2: value 68K -> 1K
- SW1: renamed from S2; value Reset -> RST; footprint 1 My Footprints:SW_Push_1P1T-SH_NO_CK_KMR2xxG_3D -> 1 My Footprints:KEY-SMD_4P-L4.2-W3.2-P2.20-LS5.1-TL
- U2: value LMR16006XDDCR -> MAX3051ESA; footprint Package_TO_SOT_SMD:SOT-23-6 -> Package_SO:SOIC-8_3.9x4.9mm_P1.27mm
- U3: value MAX3051ESA -> XC6220B331MR; footprint Package_SO:SOIC-8_3.9x4.9mm_P1.27mm -> Package_TO_SOT_SMD:SOT-23-5
- USB1: value USB-OTG -> USB; footprint Connector_USB:USB_Micro-B_Molex-105017-0001 -> 1 My Footprints:USB_Micro-B_XKB_U254-051T-4BH23-S2B
- moved R4 110.8 mm to (121.5, 82.0), turned to 90 degrees
- moved USB1 108.5 mm to (128.8, 79.8), turned to 180 degrees
- moved C9 96.9 mm to (147.4, 110.4), turned to 90 degrees
- moved D1 96.8 mm to (159.5, 83.2), turned to 0 degrees
- moved SW1 94.5 mm to (112.5, 111.0), turned to 0 degrees
- moved C11 93.4 mm to (154.8, 106.2)
- moved JP1 90.5 mm to (129.0, 103.9), turned to 180 degrees
- moved D2 83.6 mm to (122.2, 80.0), turned to 0 degrees
- moved D3 82.7 mm to (159.8, 106.6), turned to 90 degrees
- moved U3 81.4 mm to (137.9, 82.0)
- moved H2 80.8 mm to (102.5, 112.0)
- moved H3 63.8 mm to (160.0, 79.5)
- moved I2C1 59.4 mm to (141.7, 93.2)
- moved LOGO1 56.2 mm to (116.2, 107.0)
- moved J3 51.0 mm to (150.9, 80.4), turned to 180 degrees
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- renumbered C1 to C11, R6 to R4
Connections:
- net Net-(U1-Pad21) renamed /U1RX0
- net Net-(U1-Pad25) renamed /xPSRAM_CS
- net Net-(U1-Pad33) renamed /MTCK
- net Net-(U1-Pad34) renamed /MTDO
- net Net-(U1-Pad35) renamed /MTDI
- net Net-(U1-Pad36) renamed /MTMS
- net Net-(U1-Pad39) renamed /VDD_SPI
- C2 pad 1: /SW -> GND
- C2 pad 2: /CB -> +3V3
- C3 pad 1: +48V -> GND
- C3 pad 2: GND -> +3V3
- C4 pad 1: +48V -> GND
- C4 pad 2: GND -> +3V3
- C6 pad 2: +5V -> /~BOOT
- C7 pad 2: +3V3 -> /~SW_L
- C8 pad 1: +3V3 -> GND
- C8 pad 2: GND -> /~SW_S
- C9 pad 2: /~BOOT -> /~SW_R
- D1 pad 1: Net-(D4-Pad1) -> Net-(D1-Pad1)
- D2 pad 1: +5V -> Net-(D2-Pad1)
- D2 pad 2: /VBUS -> +3V3
- D3 pad 2: +5V -> GND
- D3 pad 3: Net-(D3-Pad3) -> /LED_D
- D3 pad 4: GND -> +3V3
- H1 pad 1: GNDPWR -> GND
- J2 pad 1: GND -> /U0TXD
- J2 pad 2: Net-(J2-Pad2) -> /~BOOT
- J2 pad 3: /D_TXSCL -> /U0RXD
- J2 pad 4: /D_RXSDA -> GND
- J3 pad 1: /UART_TX -> /QW_SCL
- J3 pad 2: /~BOOT -> /QW_SDA
- J3 pad 3: /UART_RX -> +3V3
- JP1 pad 1: +3V3 -> Net-(J2-Pad5)
- JP1 pad 2: /VCC_PROG -> +3V3
- JP2 pad 2: /CAN+ -> /CAN-
- R2 pad 1: /FB -> /~LED_IO2
- R2 pad 2: +5V -> Net-(D1-Pad1)
- R4 pad 2: Net-(D4-Pad1) -> Net-(D2-Pad1)
- SW1 pad 1: GND -> /~RST
- SW1 pad 2: /~RST -> GND
- U1 pad 14: /~CAN_EN -> Net-(U1-Pad14)
- U1 pad 15: /CAN_TX -> Net-(U1-Pad15)
- U1 pad 16: /CAN_RX -> Net-(U1-Pad16)
- U1 pad 18: Net-(U1-Pad18) -> /CAN_TX
- U1 pad 19: Net-(U1-Pad19) -> /CAN_RX
- U1 pad 20: Net-(U1-Pad20) -> /~CAN_EN
- U1 pad 29: Net-(U1-Pad29) -> /~SW_L
- U1 pad 30: /LED_DAT -> /~SW_S
- U1 pad 31: /D_TXSCL -> /~SW_R
- U1 pad 32: /D_RXSDA -> /LED_D
- U1 pad 37: /UART_TX -> /U0TXD
- U1 pad 38: /UART_RX -> /U0RXD
- U1 pad 5: Net-(U1-Pad5) -> /~LED_IO2
- U1 pad 6: Net-(U1-Pad6) -> /QW_SCL
- U1 pad 7: Net-(U1-Pad7) -> /QW_SDA
- U2 pad 1: /CB -> /CAN_TX
- U2 pad 3: /FB -> +3V3
- U2 pad 4: Net-(U2-Pad4) -> /CAN_RX
- U2 pad 5: +48V -> /~CAN_EN
- U2 pad 6: /SW -> /CAN-
- U3 pad 1: /CAN_TX -> /VBUS
- U3 pad 3: +3V3 -> /VBUS
- U3 pad 4: /CAN_RX -> Net-(U3-Pad4)
- U3 pad 5: /~CAN_EN -> +3V3
Routing:
- net +3V3: track 0.00 -> 143.2 mm, vias 0 -> 3
- net /~BOOT: track 0.00 -> 54.1 mm, vias 0 -> 2
- net /~RST: track 0.00 -> 51.7 mm, vias 0 -> 1
- net GNDPWR: track 0.00 -> 42.8 mm, vias 0 -> 4
- net Net-(J2-Pad5): track 0.00 -> 25.1 mm, vias 0 -> 1
- net /CAN-: track 0.00 -> 24.8 mm, vias 0 -> 1
- net /CAN+: track 0.00 -> 20.5 mm
- net +48V: track 0.00 -> 19.9 mm
- net /~SW_R: track 0.00 -> 17.5 mm
- net /USB_D+: track 0.00 -> 17.3 mm
- net /USB_D-: track 0.00 -> 16.8 mm
- net /~CAN_EN: track 0.00 -> 16.1 mm, vias 0 -> 2
- net /CAN_RX: track 0.00 -> 15.2 mm, vias 0 -> 2
- net /~SW_L: track 0.00 -> 13.8 mm
- net /~SW_S: track 0.00 -> 13.2 mm
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- added copper zone on B.Cu, net GNDPWR
- added copper zone on F.Cu, net GNDPWR
- removed copper zone on B.Cu, net +3V3
- removed copper zone on F.Cu, net +3V3
- removed copper zone on F.Cu, net +48V
- removed copper zone on F.Cu, net +5V
- removed copper zone on F.Cu, net /SW
Other:
- board size 80 x 35 mm -> 62.5 x 37.5 mm

Commit message: updoot, new rev
Parts:
- removed D1: IO2, 1 My Footprints:LED_0603_1608Metric_SnapModel
- removed R2: 1K, Resistor_SMD:R_0402_1005Metric
- D2: footprint 1 My Footprints:LED_0603_1608Metric_SnapModel -> 10-My-Footprints:LED_0603_1608Metric_SnapModel
- D3: footprint 1 My Footprints:LED_SK6812MINI_PLCC4_3.5x3.5mm_P1.75mm_3D -> 10-My-Footprints:LED_SK6812MINI_PLCC4_3.5x3.5mm_P1.75mm_3D
- I2C1: footprint 1 My Footprints:OLED_SSD1315_128x64_1.3_I2C_New_Silhouette_Big3D -> 10-My-Footprints:OLED_SSD1315_128x64_1.3_I2C_New_Silhouette_Big3D
- J2: value Conn_01x06 -> ESP-PROG; footprint ESP32-S2-DevKit-USB-Rev-B:WU06S -> 11-My-Edits:Gecko-G125_PlusTC2030_IDCBox_2x03_P1.25mm_Vertical_3D
- J3: footprint 1 My Footprints:JST_SH_SM04B-SRSS-TB_1x04-1MP_P1.00mm_Horizontal_3D -> 10-My-Footprints:JST_SH_SM04B-SRSS-TB_1x04-1MP_P1.00mm_Horizontal_3D
- LOGO1: footprint 1 My Footprints:neggle-logo-0.12 -> 10-My-Footprints:neggle-logo-0.12
- NT1: footprint NetTie:NetTie-2_THT_Pad0.3mm -> NetTie:NetTie-2_SMD_Pad0.5mm
- PS1: footprint 1 My Footprints:Converter_DCDC_TDK-Lambda_CC3-xxxxxF-E -> 10-My-Footprints:Converter_DCDC_TDK-Lambda_CC3-xxxxxF-E
- SW1, SW2, SW3, SW4, SW5: footprint 1 My Footprints:KEY-SMD_4P-L4.2-W3.2-P2.20-LS5.1-TL -> 10-My-Footprints:KEY-SMD_4P-L4.2-W3.2-P2.20-LS5.1-TL
- U1: footprint 1 My Footprints:ESP32-S2-WROVER_and_WROOM(PCB,-I(IPEX))-Universal -> 10-My-Footprints:ESP32-S2-WROVER_and_WROOM(PCB,-I(IPEX))-Universal
- USB1: footprint 1 My Footprints:USB_Micro-B_XKB_U254-051T-4BH23-S2B -> 41-EasyEDA-Edits:MICRO-USB-SMD_U254-051T-4BH83-F1S_C397452
- moved J2 18.1 mm to (130.1, 103.6), turned to 90 degrees
- moved SW2 9.80 mm to (111.5, 112.0)
- moved C6 9.76 mm to (107.9, 112.6)
- moved R6 8.28 mm to (116.9, 112.6)
- moved SW1 8.06 mm to (120.5, 112.0)
- moved JP1 8.00 mm to (128.8, 95.9), turned to 270 degrees
- moved C4 5.22 mm to (160.0, 83.2)
- moved C9 5.21 mm to (152.1, 112.6)
- moved SW5 4.68 mm to (155.8, 112.0)
- moved C8 4.61 mm to (142.1, 112.6)
- moved NT1 4.34 mm to (116.8, 90.0), turned to 0 degrees
- moved C7 4.26 mm to (132.1, 112.6)
- moved SW4 4.20 mm to (145.8, 112.0)
- moved I2C1 4.02 mm to (145.7, 93.4)
- moved J3 4.00 mm to (154.9, 80.3)
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Connections:
- J2 pad 1: /U0TXD -> /~RST
- J2 pad 2: /~BOOT -> /VPP
- J2 pad 3: /U0RXD -> /U0TXD
- J2 pad 5: Net-(J2-Pad5) -> /U0RXD
- J2 pad 6: /~RST -> /~BOOT
- JP1 pad 1: Net-(J2-Pad5) -> +3V3
- JP1 pad 2: +3V3 -> /VPP
- U1 pad 10: /OLED_SCL -> Net-(U1-Pad10)
- U1 pad 4: Net-(U1-Pad4) -> /QW_SCL
- U1 pad 5: /~LED_IO2 -> /QW_SDA
- U1 pad 6: /QW_SCL -> Net-(U1-Pad6)
- U1 pad 7: /QW_SDA -> /OLED_SDA
- U1 pad 8: Net-(U1-Pad8) -> /OLED_SCL
- U1 pad 9: /OLED_SDA -> Net-(U1-Pad9)
Routing:
- net Net-(J2-Pad5): track 25.1 -> 0.00 mm, vias 1 -> 0
- net /LED_D: track 0.00 -> 21.9 mm, vias 0 -> 2
- net /U0RXD: track 4.27 -> 22.8 mm, vias 0 -> 1
- net +3V3: track 143.2 -> 126.9 mm, vias 3 -> 5
- net /U0TXD: track 5.91 -> 22.2 mm
- net /~BOOT: track 54.1 -> 68.6 mm, vias 2 -> 3
- net /VPP: track 0.00 -> 9.65 mm
- net /~LED_IO2: track 9.48 -> 0.00 mm, vias 2 -> 0
- net /~SW_R: track 17.5 -> 24.2 mm, vias 0 -> 2
- net GNDPWR: track 42.8 -> 37.9 mm
- net /~RST: track 51.7 -> 48.4 mm
- net /~SW_S: track 13.2 -> 15.7 mm, vias 0 -> 2
- net /CAN_TX: track 8.55 -> 10.5 mm
- net Net-(D1-Pad1): track 1.92 -> 0.00 mm
- net /CAN_RX: track 15.2 -> 17.1 mm
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- added copper zone on F.Cu, net +3V3
Other:
- board size 62.5 x 37.5 mm -> 65 x 37.5 mm
