File: EltekController/EltekController.sch (KiCad schematic (older format))
At the start: 28 parts, among them J1 CANBUS, J2 Display, J3 USB_B_Micro, Q1 UMH3N, SW1 Reset, SW2 Boot, U1 ESP32-WROOM-32E, U2 CP2104-F03-GMR, U3 TJA1051T/3/1J, U4 XC6206P332MR

Commit message: updoots
Parts:
- C2: LCSC (none) -> C52923
- Q1: LCSC (none) -> C123008
Changed lines of the file:
@@
 F 2 "Package_TO_SOT_SMD:SOT-363_SC-70-6" H 1805 4960 50  0001 C CNN
 F 3 "http://rohmfs.rohm.com/en/products/databook/datasheet/discrete/transistor/digital/emh3t2r-e.pdf" H 1950 5400 50  0001 C CNN
+F 4 "C123008" H 1800 5400 50  0001 C CNN "LCSC"
 	2    1800 5400
 	0    1    1    0
@@
 F 2 "Package_TO_SOT_SMD:SOT-363_SC-70-6" H 1205 4960 50  0001 C CNN
 F 3 "http://rohmfs.rohm.com/en/products/databook/datasheet/discrete/transistor/digital/emh3t2r-e.pdf" H 1350 5400 50  0001 C CNN
+F 4 "C123008" H 1200 5400 50  0001 C CNN "LCSC"
 	1    1200 5400
 	0    -1   1    0
@@
 F 2 "Capacitor_SMD:C_0402_1005Metric" H 7788 1850 50  0001 C CNN
 F 3 "~" H 7750 2000 50  0001 C CNN
+F 4 "C52923" H 7750 2000 50  0001 C CNN "LCSC"
 	1    7750 2000
 	-1   0    0    -1

Commit message: update it so the thing kinda works
Parts:
- J3: JLCPCB_CORRECTION (none) -> 0; 0; 90
- PS1: MANUFACTURER MEANWELL -> (none); Manufacturer (none) -> MEANWELL
- R2: MPN (none) -> 0402WGF1002TCE; PN 0402WGF1002TCE -> (none)
- U1: JLCPCB_CORRECTION (none) -> 0; 0; 270; MFG Espressif -> (none); MPN (none) -> ESP32-WROOM-32E; Manufacturer (none) -> Espressif; PN ESP32-WROOM-32E -> (none)
- U2, U3: JLCPCB_CORRECTION (none) -> 0; 0; 270
- U4: JLCPCB_CORRECTION (none) -> 0; 0; 180
Changed lines of the file:
@@
 F 3 "http://ww1.microchip.com/downloads/en/DeviceDoc/20005785A.pdf" H 3000 6950 50  0001 C CNN
 F 4 "C5446" H 3000 6950 50  0001 C CNN "LCSC"
+F 5 "0; 0; 180" H 3000 6950 50  0001 C CNN "JLCPCB_CORRECTION"
 	1    3000 6950
 	1    0    0    -1
@@
 F 2 "SnapEDA-zip:CONV_SPBW06F-12" H 2050 6750 50  0001 L BNN
 F 3 "" H 1900 7150 50  0001 L BNN
-F 4 "MEANWELL" H 2050 6650 50  0001 L BNN "MANUFACTURER"
+F 4 "" H 2050 6650 50  0001 L BNN "MANUFACTURER"
+F 5 "MEANWELL" H 1900 7150 50  0001 C CNN "Manufacturer"
 	1    1900 7150
 	1    0    0    -1
@@
 F 5 "XKB Connectivity" H 1050 1750 50  0001 C CNN "Manufacturer"
 F 6 "U254-051T-4BH23-S2B" H 1050 1750 50  0001 C CNN "MPN"
+F 7 "0; 0; 90" H 1050 1750 50  0001 C CNN "JLCPCB_CORRECTION"
 	1    1050 1750
 	1    0    0    -1
@@
 F 3 "https://www.silabs.com/documents/public/data-sheets/cp2104.pdf" H 2050 3100 50  0001 C CNN
 F 4 "C47742" H 2600 1850 50  0001 C CNN "LCSC"
+F 5 "0; 0; 270" H 2600 1850 50  0001 C CNN "JLCPCB_CORRECTION"
 	1    2600 1850
 	1    0    0    -1
@@
 F 3 "http://www.nxp.com/documents/data_sheet/TJA1051.pdf" H 2000 4000 50  0001 C CNN
 F 4 "C38695" H 2000 4000 50  0001 C CNN "LCSC"
+F 5 "0; 0; 270" H 2000 4000 50  0001 C CNN "JLCPCB_CORRECTION"
 	1    2000 4000
 	1    0    0    -1
@@
 F 3 "" H 8000 1200 50  0001 C CNN
 F 4 "C25744" H 8000 1200 50  0001 C CNN "LCSC"
-F 5 "0402WGF1002TCE" H 8000 1200 50  0001 C CNN "PN"
+F 5 "" H 8000 1200 50  0001 C CNN "PN"
+F 6 "0402WGF1002TCE" H 8000 1200 50  0001 C CNN "MPN"
 	1    8000 1200
 	1    0    0    1
@@
 F 3 "https://www.espressif.com/sites/default/files/documentation/esp32-wroom-32d_esp32-wroom-32u_datasheet_en.pdf" H 5450 3300 50  0001 C CNN
 F 4 "C701341" H 5750 3250 50  0001 C CNN "LCSC"
-F 5 "Espressif" H 5750 3250 50  0001 C CNN "MFG"
-F 6 "ESP32-WROOM-32E" H 5750 3250 50  0001 C CNN "PN"
+F 5 "" H 5750 3250 50  0001 C CNN "MFG"
+F 6 "" H 5750 3250 50  0001 C CNN "PN"
+F 7 "0; 0; 270" H 5750 3250 50  0001 C CNN "JLCPCB_CORRECTION"
+F 8 "ESP32-WROOM-32E" H 5750 3250 50  0001 C CNN "MPN"
+F 9 "Espressif" H 5750 3250 50  0001 C CNN "Manufacturer"
 	1    5750 3250
 	1    0    0    -1

Commit message: v0.1
Parts:
- renumbered JP2 to JP1
Changed lines of the file:
@@
 $EndComp
 $Comp
-L Jumper:SolderJumper_3_Open JP2
+L Jumper:SolderJumper_3_Open JP1
 U 1 1 604C9D7D
 P 3000 5250
-F 0 "JP2" H 3000 5454 50  0000 C CNN
+F 0 "JP1" H 3000 5454 50  0000 C CNN
 F 1 "VDISP" H 3000 5363 50  0000 C CNN
 F 2 "Jumper:SolderJumper-3_P1.3mm_Open_RoundedPad1.0x1.5mm_NumberLabels" H 3000 5250 50  0001 C CNN

Commit message: Squashed commit of the following:
commit 90807526c89bbe23d0d14403179393f46968545b
Author: neg2led <4232981+neg2led@users.noreply.github.com>
Date:   Fri Feb 19 13:40:56 2021 +1100

    change vtabs

commit bdeb0cb4df280460f20d9cb7594185681e97bdea
Author: neg2led <4232981+neg2led@users.noreply.github.com>
Date:   Fri Feb 19 13:38:28 2021 +1100

    tiny tweak

commit 1e098ee4d97e67064c3c8c363f77a0e840b9e8c0
Author: neg2led <4232981+neg2led@users.noreply.github.com>
Date:   Fri Feb 19 13:37:41 2021 +1100

    almost...

commit b00c0a0b75bab0a44da9d349d5dc3fbb57f6d1e8
Author: neg2led <4232981+neg2led@users.noreply.github.com>
Date:   Fri Feb 19 01:39:59 2021 +1100

    and so it continues

reworked the whole dealio

almost...

tiny tweak

change vtabs
Parts:
- removed U4: XC6206P332MR, Package_TO_SOT_SMD:SOT-23, symbol Regulator_Linear:XC6206PxxxMR
- added C1, C2: 10uF, Capacitor_SMD:C_0603_1608Metric, symbol Device:C_Small
- added C7: 4.7uF, Capacitor_SMD:C_0402_1005Metric, symbol Device:C_Small
- added D1: B5819W, Diode_SMD:D_SOD-123, symbol Device:D_Schottky_Small_ALT
- added I2C1: OLED, Connector_PinSocket_2.54mm:PinSocket_1x04_P2.54mm_Vertical, symbol Connector_Generic:Conn_01x04
- added JP1: CAN_T, Jumper:SolderJumper-2_P1.3mm_Open_RoundedPad1.0x1.5mm, symbol 1_My_Symbols:SolderJumper_2_Open_Small
- added LOGO1: Logo_Open_Hardware_Small, 1 My Footprints:neggle-logo-0.12, symbol Graphic:Logo_Open_Hardware_Small
- added NT1: GND_TIE, NetTie:NetTie-2_THT_Pad0.3mm, symbol Device:Net-Tie_2
- added U4: AMS1117-3.3, Package_TO_SOT_SMD:SOT-223-3_TabPin2, symbol Regulator_Linear:AMS1117-3.3
- C3: renamed from C4; value 10uF -> 22uF; LCSC C19702 -> C59461; MPN CL10A106KP8NNNC -> CL10A226MQ8NRNC
- C4: renamed from C6; value 10uF -> 22uF; footprint Capacitor_SMD:C_0402_1005Metric -> Capacitor_SMD:C_0603_1608Metric; LCSC C15525 -> C59461; MPN CL05A106MQ5NUNC -> CL10A226MQ8NRNC
- C5: renamed from C7; value 1uF -> 100nF; footprint Capacitor_SMD:C_0402_1005Metric -> Capacitor_SMD:C_0603_1608Metric; LCSC C52923 -> C14663; MPN CL05A105KA5NQNC -> CC0603KRX7R9BB104; Manufacturer Samsung -> Yageo
- C6: renamed from C2; symbol Device:C -> Device:C_Small
- C9: renamed from C5; value 1uF -> 100nF; footprint Capacitor_SMD:C_0603_1608Metric -> Capacitor_SMD:C_0402_1005Metric; LCSC C15849 -> C1525; MPN CL10B474KA8NNNC -> CL05B104KO5NNNC
- D3: renamed from D2; value LED -> IO2
- H1, H2, H3, H4: footprint MountingHole:MountingHole_2.2mm_M2_Pad_Via -> MountingHole:MountingHole_2.7mm_M2.5_Pad_Via
- JP2: renamed from JP1; value VDISP -> VJ2
- R1: footprint Resistor_SMD:R_0402_1005Metric -> Resistor_SMD:R_0603_1608Metric_Pad0.98x0.95mm_HandSolder; LCSC C25079 -> C22787; MPN 0402WGF1200TCE -> 0603WAF1200T5E
- RN1: JLCPCB_CORRECTION (none) -> 0; 0; 90
- U1: footprint RF_Module:ESP32-WROOM-32 -> 1 My Footprints:ESP32-WROOM_WROVER_Dual_JLC_ManyVias; JLCPCB_CORRECTION 0; 0; 270 -> -3.325; 0; 0
- USB1: renamed from J3; value USB_B_Micro -> USB-SER
- renumbered C1 to C10, C3 to C8, D1 to D2, SW1 to S1, SW2 to S2
Connections:
- net labels added: CAN_S, GPIO2_LED, OLED_SCL, OLED_SDA
- net labels removed: LED_G2, RXLED, TXLED
- wire segments 167 -> 193
- no-connect marks 26 -> 32
Other:
- note added: "C6 is optional\n(for CP2102 prog. mode)"
- note added: "Display/Ext. IO"
- note added: "ESP32-WROOM-32E"
- note added: "Extra Filter"
- note added: "In Only"
- note added: "LEDs"
- note added: "MTCK"
- note added: "MTDI"
- note added: "MTDO"
- note added: "MTMS"
- note added: "Mechanical"
- note added: "PS1 is a std. SIP8 isolated DC-DC converter.\nEquivs: XP Power IZ4805S, Cincon EC4SAW-48S05N etc"
- note added: "Power Supply"
- note removed: "Board Mounts"
- note removed: "Display Connector"
- note removed: "ESP32-WROOM-32"
- note removed: "Extra Filtering"
- note removed: "GPIO2 LED"
- note removed: "Main Power & Filtering"
- note removed: "PS1 is a std. SIP8 isolated DC-DC converter.\nEquivs: XP Power IZ4805S, Cincon EC4SAW-48S05N, Recom RS6-4805S etc"
- note removed: "RGB LED"
- moved on the sheet: C10, C3, C4, C5, C6, C8, C9, D2, D3, H1, H2, H3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

Commit message: fixup ESP32 placement pos
Parts:
- U1: JLCPCB_CORRECTION -3.325; 0; 0 -> -2.875; 0; 0
Changed lines of the file:
@@
 F 3 "https://www.espressif.com/sites/default/files/documentation/esp32-wroom-32d_esp32-wroom-32u_datasheet_en.pdf" H 5700 3050 50  0001 C CNN
 F 4 "C701341" H 6000 3000 50  0001 C CNN "LCSC"
-F 5 "-3.325; 0; 0" H 6000 3000 50  0001 C CNN "JLCPCB_CORRECTION"
+F 5 "-2.875; 0; 0" H 6000 3000 50  0001 C CNN "JLCPCB_CORRECTION"
 F 6 "ESP32-WROOM-32E" H 6000 3000 50  0001 C CNN "MPN"
 F 7 "Espressif" H 6000 3000 50  0001 C CNN "Manufacturer"

Commit message: saving this because I changed my mind again
Parts:
- removed C7: 4.7uF, Capacitor_SMD:C_0402_1005Metric, symbol Device:C_Small
- removed C8: 10uF, Capacitor_SMD:C_0402_1005Metric, symbol Device:C_Small
- removed D2: RGB, 1 My Footprints:LED_RGB_2020, symbol Device:LED_RGBA
- removed PS1: SPBW06G-05, SnapEDA-zip:CONV_SPBW06F-12, symbol 1_My_Symbols:SPBW06G-05
- removed Q1: UMH3N, Package_TO_SOT_SMD:SOT-363_SC-70-6, symbol Transistor_BJT:UMH3N
- removed RN1: 1K, Resistor_SMD:R_Array_Concave_4x0402, symbol CustomDevice:R_Pack04_Split
- removed U1: ESP32-WROOM-32E, 1 My Footprints:ESP32-WROOM_WROVER_Dual_JLC_ManyVias, symbol RF_Module:ESP32-WROOM-32D
- removed U2: CP2104-F03-GMR, Package_DFN_QFN:QFN-24-1EP_4x4mm_P0.5mm_EP2.6x2.6mm, symbol Interface_USB:CP2104
- removed U3: TJA1051T/3/1J, Package_SO:SOIC-8_3.9x4.9mm_P1.27mm, symbol Interface_CAN_LIN:TJA1051T-3
- added C1: 10uF, Capacitor_SMD:C_0603_1608Metric, symbol Device:C_Small
- added C10, C9: 100nF, Capacitor_SMD:C_0402_1005Metric, symbol Device:C
- added C3: 2.2uF, Capacitor_SMD:C_1210_3225Metric_Pad1.33x2.70mm_HandSolder, symbol Device:C_Small
- added C5: 22uF, Capacitor_SMD:C_0805_2012Metric, symbol Device:C_Small
- added D1: SS210, Diode_SMD:D_PowerDI-123, symbol Device:D_Schottky_Small_ALT
- added D3: RGB, 1 My Footprints:DY-S1515065_RGBC_6805-5T, symbol 1_My_Symbols:DY-S1515065_RGBC_6805-5T
- added D4: 3V3, 1 My Footprints:LED_0603_1608Metric_SnapModel, symbol Device:LED_Small
- added J3: ESP_PROG, 1 My Footprints:JST_SH_SM06B-SRSS-TB_1x06-1MP_P1.00mm_Horizontal_3D, symbol Connector_Generic_MountingPin:Conn_01x06_MountingPin
- added JP1: VPP_EN, Jumper:SolderJumper-2_P1.3mm_Open_RoundedPad1.0x1.5mm, symbol 1_My_Symbols:SolderJumper_2_Open_Small
- added L1: 33uH, 1 My Footprints:L_Sunlord_SWPA6028S, symbol Device:L_Core_Ferrite
- added R2: 68K, Resistor_SMD:R_0402_1005Metric, symbol Device:R_Small
- added R3: 12K, Resistor_SMD:R_0402_1005Metric, symbol Device:R_Small
- added R5: 22R, Resistor_SMD:R_0402_1005Metric, symbol Device:R_Small
- added R6, R7: 1K, Resistor_SMD:R_0402_1005Metric, symbol Device:R_Small
- added U1: ESP32-S2-WROVER, 1 My Footprints:ESP32-S2-WROVER_and_WROOM(PCB,-I(IPEX))-Universal, symbol RF_Module:ESP32-S2-WROVER
- added U2: LMR16006XDDCR, Package_TO_SOT_SMD:SOT-23-6, symbol 1_My_Symbols:LMR16006XDDCR
- added U3: MAX3051ESA, Package_SO:SOIC-8_3.9x4.9mm_P1.27mm, symbol Interface_UART:MAX3051
- C12: renamed from C5; Note (none) -> 50V
- C2: value 10uF -> 100nF; footprint Capacitor_SMD:C_0603_1608Metric -> Capacitor_SMD:C_0402_1005Metric; LCSC C19702 -> C1525; MPN CL05A106MQ5NUNC -> CL05B104KO5NNNC; Note (none) -> 16V
- C4: renamed from C10; value 1uF -> 2.2uF; footprint Capacitor_SMD:C_1206_3216Metric -> Capacitor_SMD:C_1210_3225Metric_Pad1.33x2.70mm_HandSolder; LCSC C13832 -> C76685; MPN CL31B105KCHNNNE -> C3225X7R2A225KT0L0U; Manufacturer Samsung -> TDK
- C6: value 1uF -> 22uF; footprint Capacitor_SMD:C_0402_1005Metric -> Capacitor_SMD:C_0805_2012Metric; LCSC C52923 -> C45783; MPN (none) -> CL21A226MAQNNNE; Manufacturer (none) -> Samsung
- D2: renamed from D1; Manufacturer (none) -> CJ Electronics Tech; Mfg CJ Electronics Tech -> (none)
- D5: renamed from D3; value IO2 -> 5V0; Color Blue -> Green; LCSC C72041 -> C72043; MPN (none) -> 19-217/GHC-YR1S2/3T; Manufacturer (none) -> Everlight Elec
- I2C1: footprint Connector_PinSocket_2.54mm:PinSocket_1x04_P2.54mm_Vertical -> 1 My Footprints:OLED_SSD1315_128x64_1.3_I2C_New_Silhouette
- USB1: value USB-SER -> USB-OTG
- renumbered C4 to C11, C3 to C14, C1 to C7, C9 to C8, JP1 to JP2, JP2 to JP3, R2 to R1, R1 to R4, S2 to S1, S1 to S2
Connections:
- net +3V3: now also C7.2, D4.2 (A), JP1.1 (A), U1.2 (3V3), U3.3 (VDD); no longer D5.2 (A)
- net +48V: now also C4.1, C3.1, U2.5 (VIN); no longer C4.2
- net +5V: now also C6.2, D5.2 (A), C5.2, D3.2 (VDD), L1.2, R2.2; no longer C2.2, C7.1, C8.2
- net CAN+: now also U3.7 (CANH)
- net CAN-: now also U3.6 (CANL)
- net CAN_RX: now also U1.16 (IO13), U3.4 (RXD)
- net CAN_TX: now also U1.15 (IO12), U3.1 (TXD)
- net D_RXSDA: now also U1.32 (IO38)
- net D_TXSCL: now also U1.31 (IO37)
- net GND: now also C4.2, C6.1, C7.1, C8.2, NT1.2, C1.2, C10.1, C3.2, C5.1, C9.1, D1.2 (A), D3.4 (GND), J3.4 (Pin_4), J3.MP (MountPin), R3.1, R6.1, R7.1, U1.1 (GND), U1.26 (GND), U1.42 (GND), U1.43 (GND), U2.2 (GND), U3.2 (GND), U3.8 (RS); no longer C2.1, C6.2, C7.2, NT1.1
- net GNDPWR: now also NT1.1; no longer C4.1, NT1.2
- net OLED_SCL: now also U1.10 (IO07)
- net OLED_SDA: now also U1.9 (IO06)
- net UART_RX: now also J3.3 (Pin_3), U1.38 (RXD0)
- net UART_TX: now also J3.1 (Pin_1), U1.37 (TXD0)
- net USB_D+: now also U1.23 (USB_D+)
- net USB_D-: now also U1.22 (USB_D-)
- net ~BOOT: now also C9.2, J3.2 (Pin_2), U1.3 (IO00)
- net ~RST: now also C1.1, C10.2, J3.6 (Pin_6), U1.41 (EN); no longer C6.1
- net USB_ID: now reaches USB1.4 (ID)
- net at D5.1 (K): now also R7.2
- new net: D3.1 (DIN), R5.2
- new net: D4.1 (K), R6.2
- new net CB: C2.2, U2.1 (CB)
- new net FB: R2.1, R3.2, U2.3 (FB)
- new net LED_DAT: R5.1, U1.30 (IO36)
- new net SW: C2.1, D1.1 (K), L1.1, U2.6 (SW)
- new net VCC_PROG: J3.5 (Pin_5), JP1.2 (B)
- new net ~CAN_EN: U1.14 (IO11), U3.5 (SHDN)
- new net ~DFU: U1.40 (IO46)
- no-connect marks 32 -> 8
Other:
- note added: "3.3v Linear Reg"
- note added: "5V DC-DC"
- note added: "CAN/Power In"
- note added: "ESP-PROG"
- note added: "ESP32-S2-WROVER/WROOM"
- note added: "Ext. Display"
- note added: "PSRAM CS"
- note added: "SSD13xx OLED"
- note added: "U1RX0"
- note added: "micro-USB"
- note removed: "Auto-Reset"
- note removed: "C6 is optional\n(for CP2102 prog. mode)"
- note removed: "Display/Ext. IO"
- note removed: "ESP32-WROOM-32E"
- note removed: "Extra Filter"
- note removed: "In Only"
- note removed: "PS1 is a std. SIP8 isolated DC-DC converter.\nEquivs: XP Power IZ4805S, Cincon EC4SAW-48S05N etc"
- note removed: "Power Supply"
- note removed: "USB to TTL Serial"
- moved on the sheet: C11, C12, C14, C4, C7, C8, D2, D5, H1, H2, H3, H4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

Commit message: yes, good
Parts:
- removed C10: 100nF, Capacitor_SMD:C_0402_1005Metric, symbol Device:C
- removed C12: 100nF, Capacitor_SMD:C_0603_1608Metric, symbol Device:C_Small
- removed C14: 22uF, Capacitor_SMD:C_0603_1608Metric, symbol Device:C_Small
- removed C3, C4: 2.2uF, Capacitor_SMD:C_1210_3225Metric_Pad1.33x2.70mm_HandSolder, symbol Device:C_Small
- removed C5, C6: 22uF, Capacitor_SMD:C_0805_2012Metric, symbol Device:C_Small
- removed C8: 100nF, Capacitor_SMD:C_0402_1005Metric, symbol Device:C_Small
- removed D1: SS210, Diode_SMD:D_PowerDI-123, symbol Device:D_Schottky_Small_ALT
- removed D2: B5819W, Diode_SMD:D_SOD-123, symbol Device:D_Schottky_Small_ALT
- removed D3: RGB, 1 My Footprints:DY-S1515065_RGBC_6805-5T, symbol 1_My_Symbols:DY-S1515065_RGBC_6805-5T
- removed D5: 5V0, 1 My Footprints:LED_0603_1608Metric_SnapModel, symbol Device:LED_Small
- removed J2: Display, Connector_JST:JST_XH_S4B-XH-A_1x04_P2.50mm_Horizontal, symbol Connector_Generic:Conn_01x04
- removed J3: ESP_PROG, 1 My Footprints:JST_SH_SM06B-SRSS-TB_1x06-1MP_P1.00mm_Horizontal_3D, symbol Connector_Generic_MountingPin:Conn_01x06_MountingPin
- removed JP3: VJ2, Jumper:SolderJumper-3_P1.3mm_Open_RoundedPad1.0x1.5mm_NumberLabels, symbol Jumper:SolderJumper_3_Open
- removed L1: 33uH, 1 My Footprints:L_Sunlord_SWPA6028S, symbol Device:L_Core_Ferrite
- removed R3: 12K, Resistor_SMD:R_0402_1005Metric, symbol Device:R_Small
- removed R5: 22R, Resistor_SMD:R_0402_1005Metric, symbol Device:R_Small
- removed R7: 1K, Resistor_SMD:R_0402_1005Metric, symbol Device:R_Small
- removed U2: LMR16006XDDCR, Package_TO_SOT_SMD:SOT-23-6, symbol 1_My_Symbols:LMR16006XDDCR
- removed U4: AMS1117-3.3, Package_TO_SOT_SMD:SOT-223-3_TabPin2, symbol Regulator_Linear:AMS1117-3.3
- added C1: 10uF, Capacitor_SMD:C_0402_1005Metric, symbol Device:C_Small
- added C7, C8, C9: 100nF, Capacitor_SMD:C_0402_1005Metric, symbol Device:C
- added D2: PWR, 1 My Footprints:LED_0603_1608Metric_SnapModel, symbol Device:LED_ALT
- added D3: SK6812MINI, 1 My Footprints:LED_SK6812MINI_PLCC4_3.5x3.5mm_P1.75mm_3D, symbol LED:SK6812MINI
- added J2: Conn_01x06, 1 My Footprints:WU06S, symbol Connector_Generic:Conn_01x06
- added J3: Qwiic, 1 My Footprints:JST_SH_SM04B-SRSS-TB_1x04-1MP_P1.00mm_Horizontal_3D, symbol 1_My_Symbols:Conn_Qwiic_Horizontal
- added PS1: CC3-4803SF-E, 1 My Footprints:Converter_DCDC_TDK-Lambda_CC3-xxxxxF-E, symbol 1_My_Symbols:CC3-4803SF-E
- added SW3: LEFT, 1 My Footprints:KEY-SMD_4P-L4.2-W3.2-P2.20-LS5.1-TL, symbol Switch:SW_Push
- added SW4: SEL, 1 My Footprints:KEY-SMD_4P-L4.2-W3.2-P2.20-LS5.1-TL, symbol Switch:SW_Push
- added SW5: RIGHT, 1 My Footprints:KEY-SMD_4P-L4.2-W3.2-P2.20-LS5.1-TL, symbol Switch:SW_Push
- added U3: XC6220B331MR, Package_TO_SOT_SMD:SOT-23-5, symbol Regulator_Linear:XC6220B331MR
- C2: value 100nF -> 10uF; LCSC C1525 -> C15525; MPN CL05B104KO5NNNC -> CL05A106MQ5NUNC; Note 16V -> (none)
- C3: renamed from C7; footprint Capacitor_SMD:C_0603_1608Metric -> Capacitor_SMD:C_0402_1005Metric; symbol Device:C_Small -> Device:C; LCSC C19702 -> C15525; MPN CL10A106KP8NNNC -> CL05A106MQ5NUNC
- D1: renamed from D4; value 3V3 -> IO2; symbol Device:LED_Small -> Device:LED_ALT
- H1, H2, H3, H4: footprint MountingHole:MountingHole_2.7mm_M2.5_Pad_Via -> MountingHole:MountingHole_2.7mm_M2.5_ISO7380_Pad_TopBottom
- I2C1: footprint 1 My Footprints:OLED_SSD1315_128x64_1.3_I2C_New_Silhouette -> 1 My Footprints:OLED_SSD1315_128x64_1.3_I2C_New_Silhouette_Big3D
- J1: footprint 1 My Footprints:Molex_Nano-Fit_105309-xx04_1x04_P2.50mm_Vertical_Horizontal_Combined -> SnapEDA-zip:TE_5-103634-3
- R2: value 68K -> 1K; LCSC C36871 -> C11702; MPN 0402WGF6802TCE -> 0402WGF1001TCE; Manufacturer (none) -> Uni-Royal
- R6: renamed from R1; Manufacturer (none) -> Uni-Royal
- R9: renamed from R4; footprint Resistor_SMD:R_0603_1608Metric_Pad0.98x0.95mm_HandSolder -> Resistor_SMD:R_0805_2012Metric_Pad1.15x1.40mm_HandSolder; LCSC C22787 -> C17437; MPN 0603WAF1200T5E -> 0805W8F1200T5E; Manufacturer Uniroyal Elec -> Uni-Royal
- SW1: renamed from S2; value Reset -> RST; footprint 1 My Footprints:SW_Push_1P1T-SH_NO_CK_KMR2xxG_3D -> 1 My Footprints:KEY-SMD_4P-L4.2-W3.2-P2.20-LS5.1-TL; LCSC C557592 -> C92589; MPN (none) -> K2-1808SN-A4SW-01; Manufacturer (none) -> Korean Hroparts Elec
- SW2: renamed from S1; value Boot -> BOOT; footprint 1 My Footprints:SW_Push_1P1T-SH_NO_CK_KMR2xxG_3D -> 1 My Footprints:KEY-SMD_4P-L4.2-W3.2-P2.20-LS5.1-TL; LCSC C557592 -> C92589; MPN (none) -> K2-1808SN-A4SW-01; Manufacturer (none) -> Korean Hroparts Elec
- U1: Manufacturer (none) -> Espressif
- U2: renamed from U3; JLCPCB_CORRECTION (none) -> 0;0;270
- USB1: value USB-OTG -> USB; footprint Connector_USB:USB_Micro-B_Molex-105017-0001 -> 1 My Footprints:USB_Micro-B_XKB_U254-051T-4BH23-S2B; JLCPCB_CORRECTION 0; 0; 90 -> 0;0;270; MPN U254-051T-4BH23-S2B -> (none); Manufacturer XKB Connectivity -> (none)
- renumbered C1 to C11, C11 to C4, C9 to C6, R6 to R4
Connections:
- net +5V is gone; now on an unnamed net: R2.2
- net CB is gone; now on net +3V3: C2.2
- net FB is gone; now on net ~LED_IO2: R2.1
- net SW is gone; now on net GND: C2.1
- net VCC_PROG is gone; now on net +3V3: JP1.2 (B)
- net +3V3: now also D2.2 (A), D3.4 (VDD), J3.3 (VCC), PS1.7 (+VOUT), U3.5 (VOUT); no longer JP1.1 (A)
- net +48V: now also PS1.1 (+VIN)
- net CAN+: now also R9.1; no longer JP2.2 (B)
- net CAN-: now also JP2.2 (B); no longer R9.1
- net CAN_RX: now also U1.19 (IO16); no longer U1.16 (IO13)
- net CAN_TX: now also U1.18 (IO15); no longer U1.15 (IO12)
- net GND: now also H1.1, SW1.2, SW2.2, C1.1, C7.1, C8.1, C9.1, D3.2 (VSS), J2.4 (Pin_4), J3.4 (GND), J3.MP (MountPin), PS1.5 (-VOUT), SW3.2, SW4.2, SW5.2, U3.2 (GND); no longer SW1.1, SW2.1
- net GNDPWR: now also PS1.2 (RC), PS1.3 (-VIN), PS1.MP (CASE); no longer H1.1
- net VBUS: now also C1.2, U3.1 (VIN), U3.3 (CE)
- net ~BOOT: now also SW2.1, J2.2 (Pin_2); no longer SW2.2
- net ~CAN_EN: now also U1.20 (IO17); no longer U1.14 (IO11)
- net ~RST: now also SW1.1, J2.6 (Pin_6); no longer SW1.2
- net U1RX0: now reaches U1.21 (IO18)
- net xPSRAM_CS: now reaches U1.25 (IO26)
- net ~SW_L: now reaches U1.29 (IO35)
- net ~SW_L: now also C7.2, SW3.1
- net MTCK: now reaches U1.33 (IO39)
- net MTDO: now reaches U1.34 (IO40)
- net MTDI: now reaches U1.35 (IO41)
- net MTMS: now reaches U1.36 (IO42)
- net VDD_SPI: now reaches U1.39 (IO45)
- net ~LED_IO2: now reaches U1.5 (IO02)
- net QW_SCL: now reaches U1.6 (IO03)
- net QW_SCL: now also J3.1 (SCL)
- net QW_SDA: now reaches U1.7 (IO04)
- net QW_SDA: now also J3.2 (SDA)
- net at D1.1 (K): no longer R4.2
- net D_RXSDA renamed LED_D
- net LED_D: now also D3.3 (DIN)
- net D_TXSCL renamed ~SW_R
- net ~SW_R: now also C9.2, SW5.1
- net LED_DAT renamed ~SW_S
- net ~SW_S: now also C8.2, SW4.1
- net UART_RX renamed U0RXD
- net U0RXD: now also J2.3 (Pin_3)
- net UART_TX renamed U0TXD
- net U0TXD: now also J2.1 (Pin_1)
- new net: J2.5 (Pin_5), JP1.1 (A)
- new net: D2.1 (K), R4.2
- no-connect marks 8 -> 23
Other:
- note added: "(Olimex compatible)"
- note added: "3.3V DC-DC"
- note added: "Qwiic, for reasons"
- note added: "UART/ESP-PROG"
- note added: "USB-C + Vbus Reg"
- note added: "just a little filtering,\nas a treat"
- note removed: "3.3v Linear Reg"
- note removed: "5V DC-DC"
- note removed: "ESP-PROG"
- note removed: "Ext. Display"
- note removed: "MTCK"
- note removed: "MTDI"
- note removed: "MTDO"
- note removed: "MTMS"
- note removed: "PSRAM CS"
- note removed: "U1RX0"
- note removed: "micro-USB"
- moved on the sheet: C11, C3, C4, C6, H1, H2, H3, H4, I2C1, J1, JP2, NT1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

Commit message: updoot, new rev
Parts:
- removed D1: IO2, 1 My Footprints:LED_0603_1608Metric_SnapModel, symbol Device:LED_ALT
- removed J2: Conn_01x06, 1 My Footprints:WU06S, symbol Connector_Generic:Conn_01x06
- removed JP1: VPP_EN, Jumper:SolderJumper-2_P1.3mm_Open_RoundedPad1.0x1.5mm, symbol 1_My_Symbols:SolderJumper_2_Open_Small
- removed R2: 1K, Resistor_SMD:R_0402_1005Metric, symbol Device:R_Small
- added J2: ESP-PROG, 11-My-Edits:Gecko-G125_PlusTC2030_IDCBox_2x03_P1.25mm_Vertical_3D, symbol Connector_Generic:Conn_02x03_Odd_Even
- added JP1: VPP_EN, Jumper:SolderJumper-2_P1.3mm_Open_RoundedPad1.0x1.5mm, symbol Device:Jumper_NO_Small
- D2: footprint 1 My Footprints:LED_0603_1608Metric_SnapModel -> 10-My-Footprints:LED_0603_1608Metric_SnapModel
- D3: footprint 1 My Footprints:LED_SK6812MINI_PLCC4_3.5x3.5mm_P1.75mm_3D -> 10-My-Footprints:LED_SK6812MINI_PLCC4_3.5x3.5mm_P1.75mm_3D
- I2C1: footprint 1 My Footprints:OLED_SSD1315_128x64_1.3_I2C_New_Silhouette_Big3D -> 10-My-Footprints:OLED_SSD1315_128x64_1.3_I2C_New_Silhouette_Big3D
- J3: footprint 1 My Footprints:JST_SH_SM04B-SRSS-TB_1x04-1MP_P1.00mm_Horizontal_3D -> 10-My-Footprints:JST_SH_SM04B-SRSS-TB_1x04-1MP_P1.00mm_Horizontal_3D
- LOGO1: footprint 1 My Footprints:neggle-logo-0.12 -> 10-My-Footprints:neggle-logo-0.12
- NT1: footprint NetTie:NetTie-2_THT_Pad0.3mm -> NetTie:NetTie-2_SMD_Pad0.5mm
- PS1: footprint 1 My Footprints:Converter_DCDC_TDK-Lambda_CC3-xxxxxF-E -> 10-My-Footprints:Converter_DCDC_TDK-Lambda_CC3-xxxxxF-E
- SW1, SW2, SW3, SW4, SW5: footprint 1 My Footprints:KEY-SMD_4P-L4.2-W3.2-P2.20-LS5.1-TL -> 10-My-Footprints:KEY-SMD_4P-L4.2-W3.2-P2.20-LS5.1-TL
- U1: footprint 1 My Footprints:ESP32-S2-WROVER_and_WROOM(PCB,-I(IPEX))-Universal -> 10-My-Footprints:ESP32-S2-WROVER_and_WROOM(PCB,-I(IPEX))-Universal
- USB1: footprint 1 My Footprints:USB_Micro-B_XKB_U254-051T-4BH23-S2B -> 41-EasyEDA-Edits:MICRO-USB-SMD_U254-051T-4BH83-F1S_C397452; LCSC C319164 -> C397452
Connections:
- net ~LED_IO2 is gone; now on net QW_SDA: U1.5 (IO02)
- net +3V3: now also JP1.1
- net GND: now also J2.4 (Pin_4)
- net OLED_SCL: now also U1.8 (IO05); no longer U1.10 (IO07)
- net OLED_SDA: now also U1.7 (IO04); no longer U1.9 (IO06)
- net QW_SCL: now also U1.4 (IO01); no longer U1.6 (IO03)
- net QW_SDA: no longer U1.7 (IO04)
- net U0RXD: now also J2.5 (Pin_5)
- net U0TXD: now also J2.3 (Pin_3)
- net ~BOOT: now also J2.6 (Pin_6)
- net ~RST: now also J2.1 (Pin_1)
- new net VPP: J2.2 (Pin_2), JP1.2
- no-connect marks 23 -> 14
Other:
- note removed: "(Olimex compatible)"
- moved on the sheet: D2, D3, R4
