File: boards/EltekController-panel.kicad_pcb (KiCad board)
At the start: 2 copper layers, 75 x 90 mm, 153 parts, among them J1 CANBUS, J2 ESP-PROG, J3 Qwiic, SW1 RST, SW2 BOOT, SW3 LEFT, SW4 SEL, SW5 RIGHT, U1 ESP32-S2-WROVER, U2 MAX3051ESA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

Commit message: Deploying to gh-pages from @ neg2led/esp32-cantroller@9e89654d6dfeae13c7be468706d1b1205d629a69 🚀
Parts:
- removed the J1 at (62.5, 103.5)
- removed the JP1 at (78.8, 109.4)
- removed the REF** at (55.0, 131.5) (x2)
- removed the REF** at (110.0, 46.5) (x2)
- removed the REF** at (55.0, 46.5) (x2)
- added REF**: NPTH, NPTH, F.Cu at (91.8, 90.8)
- added REF**: NPTH, NPTH, F.Cu at (73.2, 87.3)
- added REF**: Fiducial, Fiducial, B.Cu at (55.0, 131.5)
- added REF**: Fiducial, Fiducial, F.Cu at (55.0, 131.5)
- added REF**: Fiducial, Fiducial, B.Cu at (110.0, 46.5)
- added REF**: Fiducial, Fiducial, F.Cu at (110.0, 46.5)
- added REF**: Fiducial, Fiducial, B.Cu at (55.0, 46.5)
- added REF**: Fiducial, Fiducial, F.Cu at (55.0, 46.5)
- J1: renamed from REF**; value NPTH -> CANBUS; footprint NPTH -> 11-My-Edits:Molex_Nano-Fit_105313-xx04_1x04_P2.50mm_Horizontal_3D
- JP1: renamed from REF**; value NPTH -> VPP_EN; footprint NPTH -> Jumper:SolderJumper-2_P1.3mm_Open_RoundedPad1.0x1.5mm
- moved J1 32.0 mm to (62.5, 103.5)
- moved JP1 22.8 mm to (78.8, 109.4), turned to 270 degrees

Commit message: Deploying to gh-pages from @ neg2led/esp32-cantroller@bba46f7c44b3983ce4b2cce59a1c126a2482bb3f 🚀
Parts:
- removed the H3 at (112.5, 93.0)
- removed the H3 at (112.5, 52.5)
- removed the REF** at (55.0, 131.5) (x2)
- removed the REF** at (110.0, 46.5) (x2)
- removed the REF** at (55.0, 46.5) (x2)
- removed the U3 at (86.9, 94.4)
- removed the U3 at (86.9, 53.9)
- added C7: 100nF, Capacitor_SMD:C_0402_1005Metric, F.Cu at (82.1, 126.1)
- added C7: 100nF, Capacitor_SMD:C_0402_1005Metric, F.Cu at (82.1, 85.6)
- added PS1: CC3-4803SF-E, 10-My-Footprints:Converter_DCDC_TDK-Lambda_CC3-xxxxxF-E, F.Cu at (63.8, 114.0)
- added PS1: CC3-4803SF-E, 10-My-Footprints:Converter_DCDC_TDK-Lambda_CC3-xxxxxF-E, F.Cu at (63.8, 73.5)
- added REF**: Fiducial, Fiducial, B.Cu at (55.0, 131.5)
- added REF**: Fiducial, Fiducial, F.Cu at (55.0, 131.5)
- added REF**: Fiducial, Fiducial, B.Cu at (110.0, 46.5)
- added REF**: Fiducial, Fiducial, F.Cu at (110.0, 46.5)
- added REF**: Fiducial, Fiducial, B.Cu at (55.0, 46.5)
- added REF**: Fiducial, Fiducial, F.Cu at (55.0, 46.5)
- H3 (x2): renamed from C7; value 100nF -> MP; footprint Capacitor_SMD:C_0402_1005Metric -> MountingHole:MountingHole_2.7mm_M2.5_ISO7380_Pad_TopBottom
- U3 (x2): renamed from PS1; value CC3-4803SF-E -> XC6220B331MR; footprint 10-My-Footprints:Converter_DCDC_TDK-Lambda_CC3-xxxxxF-E -> Package_TO_SOT_SMD:SOT-23-5
- moved H3 44.9 mm to (112.5, 52.5), turned to 180 degrees
- moved H3 44.9 mm to (112.5, 93.0), turned to 180 degrees
- moved U3 30.3 mm to (86.9, 94.4), turned to 270 degrees
- moved U3 30.3 mm to (86.9, 53.9), turned to 270 degrees
Connections:
- U3 pad 1: Board_2-Board_1-+48V -> Board_2-Board_1-/VBUS
- U3 pad 2: Board_2-Board_1-GNDPWR -> Board_2-Board_1-GND
- U3 pad 3: Board_2-Board_1-GNDPWR -> Board_2-Board_1-/VBUS
- U3 pad 4: Board_2-Board_1-Net-(PS1-Pad4) -> Board_2-Board_1-Net-(U3-Pad4)
- U3 pad 5: Board_2-Board_1-GND -> Board_2-Board_1-+3V3
- U3 pad 1: Board_1-Board_1-+48V -> Board_1-Board_1-/VBUS
- U3 pad 2: Board_1-Board_1-GNDPWR -> Board_1-Board_1-GND
- U3 pad 3: Board_1-Board_1-GNDPWR -> Board_1-Board_1-/VBUS
- U3 pad 4: Board_1-Board_1-Net-(PS1-Pad4) -> Board_1-Board_1-Net-(U3-Pad4)
- U3 pad 5: Board_1-Board_1-GND -> Board_1-Board_1-+3V3
