File: boards/EltekController.kicad_pcb (KiCad board)
At the start: 2 copper layers, 65 x 37.5 mm, 36 parts, among them J1 CANBUS, J2 ESP-PROG, J3 Qwiic, SW1 RST, SW2 BOOT, SW3 LEFT, SW4 SEL, SW5 RIGHT, U1 ESP32-S2-WROVER, U2 MAX3051ESA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

Commit message: Deploying to gh-pages from @ neg2led/esp32-cantroller@bba46f7c44b3983ce4b2cce59a1c126a2482bb3f 🚀
Parts:
- removed the C3 at (141.8, 94.2)
- removed the C8 at (159.6, 116.9)
- added H2: MP, MountingHole:MountingHole_2.7mm_M2.5_ISO7380_Pad_TopBottom, F.Cu at (120.0, 116.2)
- added SW2: BOOT, 10-My-Footprints:KEY-SMD_4P-L4.2-W3.2-P2.20-LS5.1-TL, F.Cu at (129.0, 116.2)
- C3: renamed from H2; value MP -> 10uF; footprint MountingHole:MountingHole_2.7mm_M2.5_ISO7380_Pad_TopBottom -> Capacitor_SMD:C_0402_1005Metric
- C8: renamed from SW2; value BOOT -> 100nF; footprint 10-My-Footprints:KEY-SMD_4P-L4.2-W3.2-P2.20-LS5.1-TL -> Capacitor_SMD:C_0402_1005Metric
- moved C3 31.0 mm to (141.8, 94.2)
- moved C8 30.6 mm to (159.6, 116.9), turned to 90 degrees
Connections:
- C8 pad 1: Board_1-/~BOOT -> Board_1-GND
- C8 pad 2: Board_1-GND -> Board_1-/~SW_S
